File: schematics/microphone_pelican.kicad_sch (KiCad schematic)
At the start: 4 parts

Commit message: pushed place
Parts:
- C501: LCSC Part # C71629 -> C1525
- C502: LCSC Part # C76999 -> C52923
Changed lines of the file:
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@@
 			)
 		)
-		(property "LCSC Part #" "C71629"
+		(property "LCSC Part #" "C1525"
 			(at 92.71 59.69 0)
 			(hide yes)
@@
 			)
 		)
-		(property "LCSC Part #" "C76999"
+		(property "LCSC Part #" "C52923"
 			(at 119.38 62.23 0)
 			(hide yes)
