File: schematics/power_pelican.kicad_sch (KiCad schematic)
At the start: 43 parts, among them Q201 NDS7002A, Q202 DMG2305UX-13, Q203 DMG2305UX-13, Q204 NDS7002A

Commit message: Pre-layout schematic cleanup: net-naming pass + clear all ERC errors
Net naming (role-token scheme): BAT_V_STAT->VBAT_SNS,
BAT_CHG_STAT->CHG_STAT_N, BAT_CHG_SRC_STAT->CHG_IN_VLD_N,
HOLD_PWR->PWR_HOLD, CAM_RESET->CAM_RST_N (bus alias updated), and the
PWR_SRC->PWR_SRC_STAT mux-status fix. Plus in-progress storage/ethernet/
usb sheet edits and removal of the stale exported PDF.

ERC error fixes (9 -> 0):
- PWR_FLAG on the four undriven power nets (GND, GNDUSB, GNDETH,
  VBAT_GATE); PWR_FLAG added to the project power symbol library
- Ground SoC codec pin 32 (CODEC_MIC0N); MIC0_N kept as a GND alias
- Redundant paralleled power pins modeled as passive so ERC no longer
  reports power-output conflicts (TPS2116 VOUT, BQ24074 OUT/BAT, USB-C
  VBUS) - source symbols and embedded copies both updated
- JTAG_TP301/302 assigned a bare test pad (testpoint:TestPoint_Pad_D1.5mm),
  new project testpoint footprint library registered

Remaining 68 ERC items are all warnings: footprint-filter mismatches,
SPICE-model notes, and the two intentional MIC0_N=GND aliases.
Connections:
- net BAT_CHG_SRC_STAT renamed CHG_IN_VLD_N
- net BAT_CHG_STAT renamed CHG_STAT_N
- net BAT_V_STAT renamed VBAT_SNS
- net HOLD_PWR renamed PWR_HOLD
- net PWR_SRC renamed PWR_SRC_STAT
Changed lines of the file:
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@@
 		)
 	)
-	(global_label "BAT_CHG_SRC_STAT"
+	(global_label "CHG_IN_VLD_N"
 		(shape output)
 		(at 295.91 82.55 180)
@@
 		)
 	)
-	(global_label "BAT_V_STAT"
+	(global_label "VBAT_SNS"
 		(shape output)
 		(at 166.37 86.36 0)
@@
 		)
 	)
-	(global_label "BAT_CHG_STAT"
+	(global_label "CHG_STAT_N"
 		(shape output)
 		(at 312.42 82.55 0)
@@
 		)
 	)
-	(global_label "HOLD_PWR"
+	(global_label "PWR_HOLD"
 		(shape input)
 		(at 114.3 118.11 180)
@@
 		)
 	)
-	(global_label "PWR_SRC"
+	(global_label "PWR_SRC_STAT"
 		(shape input)
 		(at 185.42 170.18 180)
@@
 		)
 		(property "Intersheetrefs" "${INTERSHEET_REFS}"
-			(at 173.7263 170.18 0)
+			(at 168.5254 170.18 0)
 			(hide yes)
 			(show_name no)
@@
 		)
 	)
-	(global_label "PWR_SRC"
+	(global_label "PWR_SRC_STAT"
 		(shape input)
 		(at 173.99 185.42 0)
@@
 		)
 		(property "Intersheetrefs" "${INTERSHEET_REFS}"
-			(at 185.6837 185.42 0)
+			(at 190.8846 185.42 0)
 			(hide yes)
 			(show_name no)
@@
 					(unit 1)
 				)
+			)
+		)
+	)
+	(symbol
+		(lib_id "power:PWR_FLAG")
+		(at 124.46 177.8 0)
+		(unit 1)
+		(exclude_from_sim no)
+		(in_bom yes)
+		(on_board yes)
+		(dnp no)
+		(fields_autoplaced yes)
+		(property "Reference" "#FLG0201"
+			(at 124.46 173.99 0)
+			(hide yes)
+			(effects
+				(font
+					(size 1.27 1.27)
+				)
+			)
+		)
+		(property "Value" "PWR_FLAG"
+			(at 124.46 181.61 0)
+			(effects
+				(font
+					(size 1.27 1.27)
+				)
+			)
+		)
+		(property "Footprint" ""
+			(at 124.46 177.8 0)
+			(hide yes)
+			(effects
+				(font
+					(size 1.27 1.27)
+				)
+			)
+		)
+		(property "Datasheet" ""
+			(at 124.46 177.8 0)
+			(hide yes)
+			(effects
+				(font
+					(size 1.27 1.27)
+				)
+			)
+		)
+		(pin "1"
+		)
+		(instances
+			(project "pelican"
+				(path "/03ccc822-2fac-4029-af97-539e9460fe35/3345064e-ebc3-49d0-bdab-fd2c2db56ccd"
+					(reference "#FLG0201")
+					(unit 1)
+				)

Commit message: pushed place
Parts:
- removed BAT_J201, SW_J202: 436500200, J_436500200:J_436500200, symbol J_436500200:436500200
- added CN201: 43045-0401, J_43045-0401:J_43045-0401_2x02_RA, symbol J_43045-0401:43045-0401
- BAT_LED201: value LTST-C193KGKT-5A -> APTD1608CGCK; LCSC Part # C125102 -> C5121471
- C203, C204, C206: LCSC Part # C71629 -> C1525
- C207, C211, C212: LCSC Part # C71633 -> C19666
- C210: LCSC Part # C76999 -> C52923
- R201: value 100K -> 10K; symbol R_RC0402FR:RC0402FR-07100KL -> R_RC0402FR:RC0402FR-0710KL; LCSC Part # C60490 -> C25744
- R202, R208: LCSC Part # C106232 -> C25076
- R203, R204, R205, R207, R210, R212, R214, R215: LCSC Part # C60491 -> C25741
- R206: LCSC Part # C114763 -> C25764
- R211, R218, R219, R220: LCSC Part # C60490 -> C25744
Connections:
- net GND: now also CN201.2, CN201.4
- net SW_STAT: now also CN201.3
- net VBAT: now also CN201.1
Other:
- moved on the sheet: BAT_LED201, Q201, Q202, Q203, Q204, R201, R202, R203, R204, R205, R206, R207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
