File: schematics/storage_pelican.kicad_sch (KiCad schematic)
At the start: 5 parts

Commit message: Pre-layout schematic cleanup: net-naming pass + clear all ERC errors
Net naming (role-token scheme): BAT_V_STAT->VBAT_SNS,
BAT_CHG_STAT->CHG_STAT_N, BAT_CHG_SRC_STAT->CHG_IN_VLD_N,
HOLD_PWR->PWR_HOLD, CAM_RESET->CAM_RST_N (bus alias updated), and the
PWR_SRC->PWR_SRC_STAT mux-status fix. Plus in-progress storage/ethernet/
usb sheet edits and removal of the stale exported PDF.

ERC error fixes (9 -> 0):
- PWR_FLAG on the four undriven power nets (GND, GNDUSB, GNDETH,
  VBAT_GATE); PWR_FLAG added to the project power symbol library
- Ground SoC codec pin 32 (CODEC_MIC0N); MIC0_N kept as a GND alias
- Redundant paralleled power pins modeled as passive so ERC no longer
  reports power-output conflicts (TPS2116 VOUT, BQ24074 OUT/BAT, USB-C
  VBUS) - source symbols and embedded copies both updated
- JTAG_TP301/302 assigned a bare test pad (testpoint:TestPoint_Pad_D1.5mm),
  new project testpoint footprint library registered

Remaining 68 ERC items are all warnings: footprint-filter mismatches,
SPICE-model notes, and the two intentional MIC0_N=GND aliases.
Parts:
- removed R602: 10K, R_RC0402FR:R_RC0402FR, symbol R_RC0402FR:RC0402FR-0710KL
- removed STORE_LED601: SZYY0402YG, LED_SZYY0402YG:LED_SZYY0402YG, symbol LED_SZYY0402YG:SZYY0402YG

Commit message: pushed place
Parts:
- C601: LCSC Part # C71629 -> C1525
- R601: LCSC Part # C60490 -> C25744
Changed lines of the file:
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@@
 			)
 		)
-		(property "LCSC Part #" "C71629"
+		(property "LCSC Part #" "C1525"
 			(at 93.98 60.96 0)
 			(hide yes)
@@
 			)
 		)
-		(property "LCSC Part #" "C60490"
+		(property "LCSC Part #" "C25744"
 			(at 73.66 58.42 0)
 			(hide yes)
