File: schematics/usb_pelican.kicad_sch (KiCad schematic)
At the start: 7 parts

Commit message: Pre-layout schematic cleanup: net-naming pass + clear all ERC errors
Net naming (role-token scheme): BAT_V_STAT->VBAT_SNS,
BAT_CHG_STAT->CHG_STAT_N, BAT_CHG_SRC_STAT->CHG_IN_VLD_N,
HOLD_PWR->PWR_HOLD, CAM_RESET->CAM_RST_N (bus alias updated), and the
PWR_SRC->PWR_SRC_STAT mux-status fix. Plus in-progress storage/ethernet/
usb sheet edits and removal of the stale exported PDF.

ERC error fixes (9 -> 0):
- PWR_FLAG on the four undriven power nets (GND, GNDUSB, GNDETH,
  VBAT_GATE); PWR_FLAG added to the project power symbol library
- Ground SoC codec pin 32 (CODEC_MIC0N); MIC0_N kept as a GND alias
- Redundant paralleled power pins modeled as passive so ERC no longer
  reports power-output conflicts (TPS2116 VOUT, BQ24074 OUT/BAT, USB-C
  VBUS) - source symbols and embedded copies both updated
- JTAG_TP301/302 assigned a bare test pad (testpoint:TestPoint_Pad_D1.5mm),
  new project testpoint footprint library registered

Remaining 68 ERC items are all warnings: footprint-filter mismatches,
SPICE-model notes, and the two intentional MIC0_N=GND aliases.
Changed lines of the file:
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@@
+		)
+	)
+	(symbol
+		(lib_id "power:PWR_FLAG")
+		(at 101.6 44.45 0)
+		(unit 1)
+		(exclude_from_sim no)
+		(in_bom yes)
+		(on_board yes)
+		(dnp no)
+		(fields_autoplaced yes)
+		(property "Reference" "#FLG0701"
+			(at 101.6 40.64 0)
+			(hide yes)
+			(effects
+				(font
+					(size 1.27 1.27)
+				)
+			)
+		)
+		(property "Value" "PWR_FLAG"
+			(at 101.6 48.260000000000005 0)
+			(effects
+				(font
+					(size 1.27 1.27)
+				)
+			)
+		)
+		(property "Footprint" ""
+			(at 101.6 44.45 0)
+			(hide yes)
+			(effects
+				(font
+					(size 1.27 1.27)
+				)
+			)
+		)
+		(property "Datasheet" ""
+			(at 101.6 44.45 0)
+			(hide yes)
+			(effects
+				(font
+					(size 1.27 1.27)
+				)
+			)
+		)
+		(pin "1"
+		)
+		(instances
+			(project "pelican"
+				(path "/03ccc822-2fac-4029-af97-539e9460fe35/676f47cc-81fa-4570-932f-1e8291c2a37f"
+					(reference "#FLG0701")
+					(unit 1)
+				)
+			)
 		)
 	)

Commit message: pushed place
Parts:
- removed USBC_J701: USB-C-16P, J_USB-C-16P:J_USB-C-16P_SMD, symbol J_USB-C-16P:USB-C-16P
- added USB701: USB4120-03-C, J_USB4120-03-C:J_USB4120-03-C_SMD, symbol J_USB4120-03-C:USB4120-03-C
- C701: LCSC Part # C71629 -> C1525
- R701, R702: LCSC Part # C105872 -> C25905
- R703: LCSC Part # C60491 -> C25741
- R704: LCSC Part # C114763 -> C25764
Connections:
- net GNDUSB: now also USB701.0 (SHIELD), USB701.A1 (GND1), USB701.A12 (GND3), USB701.B1 (GND2), USB701.B12 (GND4)
- net USB_ESD_N: now also USB701.A7 (DN1), USB701.B7 (DN2)
- net USB_ESD_P: now also USB701.A6 (DP1), USB701.B6 (DP2)
- net VUSB: now also USB701.A4 (VBUS1), USB701.A9 (VBUS3), USB701.B4 (VBUS2), USB701.B9 (VBUS4)
- net at R702.2: now also USB701.B5 (CC2)
- net at R701.2: now also USB701.A5 (CC1)
Other:
- moved on the sheet: C701
