File: pelican.kicad_pcb (KiCad board)
At the start: 4 copper layers, 38 x 64 mm, 91 parts, among them CN201 43045-0401, J801 HR911105A, Q201 NDS7002A, Q202 DMG2305UX-13, Q203 DMG2305UX-13, Q204 NDS7002A, Q401 NDS7002A

Commit message: pushed pcb routing
Parts:
- C701, R701, R702: moved to F.Cu
- moved C501 33.0 mm to (222.5, 86.0)
- moved C502 33.0 mm to (223.0, 84.0)
- moved R501 33.0 mm to (221.8, 84.0)
- moved BAT_LED201 25.9 mm to (215.0, 118.0)
- moved MIC_M501 24.2 mm to (219.0, 89.8)
- moved R403 20.9 mm to (197.4, 95.2), turned to 180 degrees
- moved PROG_SW302 16.6 mm to (198.9, 125.5), turned to -90 degrees
- moved Q204 14.6 mm to (213.5, 121.5), turned to 0 degrees
- moved RESET_SW301 12.4 mm to (217.2, 130.7), turned to -90 degrees
- moved R208 12.1 mm to (216.5, 117.8), turned to -90 degrees
- moved ALIVE_LED301 11.0 mm to (199.3, 119.1), turned to 180 degrees
- moved R704 10.1 mm to (216.0, 104.5)
- moved R305 10.0 mm to (189.0, 133.5)
- moved R301 9.53 mm to (197.1, 119.1)
- moved R401 9.42 mm to (186.5, 114.4)
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Connections:
- C202 pad 1: Net-(C202-Pad1) -> VBAT_GATE
- C204 pad 1: Net-(C202-Pad1) -> VBAT_GATE
Routing:
- net VCC_3V3: track 0.00 -> 122.7 mm, vias 0 -> 6
- net GND: track 0.00 -> 93.7 mm, vias 0 -> 38
- net VUSB: track 0.00 -> 64.2 mm, vias 0 -> 7
- net CHG_STAT_N: track 0.00 -> 52.8 mm, vias 0 -> 1
- net PWR_SRC_STAT: track 1.50 -> 49.0 mm
- net LED_BAT: track 0.00 -> 31.4 mm, vias 0 -> 1
- net /Core/JTAG_TMS: track 0.00 -> 28.1 mm, vias 0 -> 1
- net SW_STAT: track 4.50 -> 32.5 mm, vias 0 -> 1
- net /Core/JTAG_TCK: track 0.00 -> 26.1 mm, vias 0 -> 1
- net VCC_5V0: track 0.00 -> 25.1 mm, vias 0 -> 2
- net /USB/USB_ESD_N: track 0.00 -> 22.5 mm, vias 0 -> 2
- net /USB/USB_ESD_P: track 0.00 -> 22.5 mm, vias 0 -> 2
- net /Core/RESET_N: track 0.00 -> 21.8 mm, vias 0 -> 1
- net PWR_HOLD: track 1.68 -> 22.8 mm, vias 0 -> 1
- net VBAT: track 0.00 -> 20.4 mm
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- added copper zone on In1.Cu, net GND
- added copper zone on In1.Cu, net GNDETH
- added copper zone on In1.Cu, net GNDUSB
- added copper zone on F.Cu, net VBAT
Other:
- board text removed: "For Instructional Use Only."
- board text removed: "SOLIDWORKS Educational Product."
